Commit message: New urdf + mesh

File: Mechanical/V3/V3_3/urdf_mesh/Base_shoulder_forearm_comined/urdf/Base_shoulder_forearm_comined.urdf (robot description, URDF)
Before this commit: robot Base_shoulder_forearm_comined, 5 links, 4 joints
Links:
- link Link_1: geometry collision mesh filename=package://Base_shoulder_forearm_combined/meshes/Link_1_coli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; visual mesh filename=package://Base_shoulder_forearm_combined/meshes/Link_1.STL
- link Link_2: geometry collision mesh filename=package://Base_shoulder_forearm_combined/meshes/Link_2_coli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; visual mesh filename=package://Base_shoulder_forearm_combined/meshes/Link_2.STL
- link Link_3: geometry collision mesh filename=package://Base_shoulder_forearm_combined/meshes/Link_3_coli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; visual mesh filename=package://Base_shoulder_forearm_combined/meshes/Link_3.STL
- link Link_4: geometry collision mesh filename=package://Base_shoulder_forearm_combined/meshes/Link_4_coli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; visual mesh filename=package://Base_shoulder_forearm_combined/meshes/Link_4.STL
- link base_link: geometry collision mesh filename=package://Base_shoulder_forearm_combined/meshes/base_link_c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; visual mesh filename=package://Base_shoulder_forearm_combined/meshes/base_link.S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
