File: Electrical/driver_board/driver_board_v2/driver_board/untitled.kicad_sch (KiCad schematic)
At the start: 28 parts, among them J1 USB_C_Receptacle_USB2.0_14P, U1 AMS1117-3.3

Commit message: Improved routing
Parts:
- removed C1, C?: 4,7u, symbol Device:C
- removed C2, C3: C, symbol Device:C
- removed C? (x2): 15pF, symbol Device:C
- removed C? (x4): 100nF, symbol Device:C
- removed C? (x2): 1µF, symbol Device:C
- removed C?: 0.1µF, symbol Device:C
- removed C?: 10nF, symbol Device:C
- removed D1: LED, symbol Device:LED
- removed FB?: FerriteBead, symbol Device:FerriteBead
- removed J1: USB_C_Receptacle_USB2.0_14P, symbol Connector:USB_C_Receptacle_USB2.0_14P
- removed J?: Conn_01x04_Pin, symbol Connector:Conn_01x04_Pin
- removed R1, R2: R, symbol Device:R
- removed R3, R4: 1.5kΩ, symbol Device:R
- removed R?: 200Ω, symbol Device:R
- removed SW?: SW_Push, symbol Switch:SW_Push
- removed SW?: SW_SPDT, symbol Switch:SW_SPDT
- removed U1: AMS1117-3.3, Package_TO_SOT_SMD:SOT-223-3_TabPin2, symbol Regulator_Linear:AMS1117-3.3
- removed U?: STM32F446RETx, Package_QFP:LQFP-64_10x10mm_P0.5mm, symbol MCU_ST_STM32F4:STM32F446RETx
- removed Y?: 8Mhz, symbol Device:Crystal
