File: Electrical/driver_board/driver_board_v2/driver_board/_autosave-microcontroller.kicad_sch (KiCad schematic)
At the start: 28 parts, among them J1 USB_C_Receptacle_USB2.0_14P, U1 AMS1117-3.3

Commit message: Update to circuit
Parts:
- gave numbers to parts that had none: 15
- renumbered C2 to C13, C3 to C14, R4 to R2
Other:
- moved on the sheet: C12, C9, J?, R1
