File: Electrical/driver_board/driver_board_v2/driver_board/driver_board.kicad_sch (KiCad schematic)
At the start: 0 parts

Commit message: Pull up/downs
Other:
- added sheet Pull resistors (pull-resistors.kicad_sch)
Changed lines of the file:
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@@
+	)
+	(sheet
+		(at 177.8 101.6)
+		(size 43.18 20.32)
+		(exclude_from_sim no)
+		(in_bom yes)
+		(on_board yes)
+		(dnp no)
+		(fields_autoplaced yes)
+		(stroke
+			(width 0.1524)
+			(type solid)
+		)
+		(fill
+			(color 0 0 0 0)
+		)
+		(property "Sheetname" "Pull resistors"
+			(at 177.8 100.8884 0)
+			(show_name no)
+			(do_not_autoplace no)
+			(effects
+				(font
+					(size 1.27 1.27)
+				)
+				(justify left bottom)
+			)
+		)
+		(property "Sheetfile" "pull-resistors.kicad_sch"
+			(at 177.8 122.5046 0)
+			(show_name no)
+			(do_not_autoplace no)
+			(effects
+				(font
+					(size 1.27 1.27)
+				)
+				(justify left top)
+			)
+		)
+		(instances
+			(project "driver_board"
+				(path "/914a9dfd-cc72-459d-a4b5-1249c31e6215"
+					(page "7")
+				)
+			)
+		)
 	)
 	(sheet
