File: Electrical/driver_board/driver_board_v2/driver_board/microcontroller.kicad_sch (KiCad schematic)
At the start: 28 parts, among them J1 Conn_01x04_Pin, J2 USB_C_Receptacle_USB2.0_14P, SW1 SW_Push, SW2 SW_SPDT, U1 STM32F446RETx, U5 USBLC6-2SC6, Y1 8Mhz

Commit message: Pull up/downs
Parts:
- removed R17, R18: 4.7kΩ, symbol Device:R
- removed R5: 10kΩ, symbol Device:R
Connections:
- net PA10_DIR_DRV4 renamed PA10_DIR_DRV4_MCU
- net PA15_STEP_DRV2 renamed PA15_STEP_DRV2_MCU
- net PA1_CS_DRV4 renamed PA1_CS_DRV4_MCU
- net PA8_STEP_DRV1 renamed PA8_STEP_DRV1_MCU
- net PA9_DIR_DRV5 renamed PA9_DIR_DRV5_MCU
- net PB0_CS_DRV6 renamed PB0_CS_DRV6_MCU
- net PB2_DIR_DRV1 renamed PB2_DIR_DRV1_MCU
- net PB4_STEP_DRV3 renamed PB4_STEP_DRV3_MCU
- net PB6_STEP_DRV4 renamed PB6_STEP_DRV4_MCU
- net PB8_STEP_DRV6 renamed PB8_STEP_DRV6_MCU
- net PC0_CS_DRV1 renamed PC0_CS_DRV1_MCU
- net PC1_CS_DRV2 renamed PC1_CS_DRV2_MCU
- net PC2_CS_DRV3 renamed PC2_CS_DRV3_MCU
- net PC6_STEP_DRV5 renamed PC6_STEP_DRV5_MCU
- net PC7_DIR_DRV2 renamed PC7_DIR_DRV2_MCU
- net PC8_DIR_DRV3 renamed PC8_DIR_DRV3_MCU
- net PC9_DIR_DRV6 renamed PC9_DIR_DRV6_MCU
- net PD2_CS_DRV5 renamed PD2_CS_DRV5_MCU
Other:
- moved on the sheet: C1, C10, C11, C12, C13, C2, C3, C4, C5, C6, C7, C8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

Commit message: Added new converter
Parts:
- renumbered U5 to U2
Changed lines of the file:
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@@
 		(dnp no)
 		(fields_autoplaced yes)
-		(property "Reference" "#PWR076"
+		(property "Reference" "#PWR014"
 			(at 184.15 107.95 0)
 			(hide yes)
@@
 			(project "driver_board"
 				(path "/914a9dfd-cc72-459d-a4b5-1249c31e6215/465404f0-d3d7-43fb-a363-deca940ffc67"
-					(reference "#PWR076")
+					(reference "#PWR014")
 					(unit 1)
 				)
@@
 		(dnp no)
 		(fields_autoplaced yes)
-		(property "Reference" "#PWR013"
+		(property "Reference" "#PWR011"
 			(at 182.88 43.18 0)
 			(hide yes)
@@
 			(project "driver_board"
 				(path "/914a9dfd-cc72-459d-a4b5-1249c31e6215/465404f0-d3d7-43fb-a363-deca940ffc67"
-					(reference "#PWR013")
+					(reference "#PWR011")
 					(unit 1)
 				)
@@
 		(dnp no)
 		(fields_autoplaced yes)
-		(property "Reference" "#PWR017"
+		(property "Reference" "#PWR013"
 			(at 184.15 95.25 0)
 			(hide yes)
@@
 			(project "driver_board"
 				(path "/914a9dfd-cc72-459d-a4b5-1249c31e6215/465404f0-d3d7-43fb-a363-deca940ffc67"
-					(reference "#PWR017")
+					(reference "#PWR013")
 					(unit 1)
 				)
@@
 		(dnp no)
 		(fields_autoplaced yes)
-		(property "Reference" "#PWR014"
+		(property "Reference" "#PWR012"
 			(at 182.88 55.88 0)
 			(hide yes)
@@
 			(project "driver_board"
 				(path "/914a9dfd-cc72-459d-a4b5-1249c31e6215/465404f0-d3d7-43fb-a363-deca940ffc67"
-					(reference "#PWR014")
+					(reference "#PWR012")
 					(unit 1)
 				)
@@
 		(in_pos_files yes)
 		(dnp no)
-		(property "Reference" "U5"
+		(property "Reference" "U2"
 			(at 253.492 101.854 0)
 			(show_name no)
@@
 			(project "driver_board"
 				(path "/914a9dfd-cc72-459d-a4b5-1249c31e6215/465404f0-d3d7-43fb-a363-deca940ffc67"
-					(reference "U5")
-					(unit 1)
-				)
+					(reference "U2")
+					(unit 1)
+				)
