File: Electrical/driver_board/driver_board_v2/driver_board/power-supply.kicad_sch (KiCad schematic)
At the start: 24 parts, among them J3 Screw_Terminal_01x02, U2 TPS54302, U3 TPS62142, U4 TPS54302

Commit message: Value assignment and protection for driver board
Parts:
- renumbered C18 to C14, C23 to C16, C19 to C17, C13 to C18, C21 to C19, C14 to C20, C20 to C21, C24 to C23, C16 to C24, C17 to C25, R8 to R6, R6 to R7, R7 to R8, U4 to U3, U3 to U4

Commit message: Added new converter
Parts:
- removed C15: 3.3uF, symbol Device:C
- removed C18: 100nF, symbol Device:C
- removed C20: 82pF, symbol Device:C
- removed C24, C25: 47uF, symbol Device:C
- removed L1: 10uH, symbol Device:L
- removed R7: 100kOhm, symbol Device:R
- removed R8: 13.7kOhm, symbol Device:R
- removed U2: TPS54302, Package_TO_SOT_SMD:SOT-23-6, symbol Regulator_Switching:TPS54302
- added Cb_inpflt1, Cb_inpflt2, Cb_inpflt3, Cb_inpflt4: 15uF, symbol Device:C
- added Cf_inpflt1: 4.7uF, symbol Device:C
- added Cff1: 8.2pF, symbol Device:C
- added Cin2, Cin5: 10uF, symbol Device:C
- added Cldo1: 1uF, symbol Device:C
- added Cout1, Cout2: 47uF, symbol Device:C
- added Lf_inpflt1: 270nH, Relay_THT:Relay_DPDT_Finder_30.22, symbol Device:L
- added Rd_inpflt1: 100mOhm, symbol Device:R
- added Rfbb1: 10kOhm, symbol Device:R
- added Rfbt1: 40.2kOhm, symbol Device:R
- added Rt1: 12.1kOhm, symbol Device:R
- added U5: TLVM13660RDLR, B3QFN20_RDL_TEX, symbol 2026-10-20_08-26-24:TLVM13660RDLR
- renumbered C16 to C15, C17 to C16, C19 to C17, C21 to C18, C22 to C19, C23 to C20, L2 to L1, L3 to L2, R6 to R5, R9 to R6, R10 to R7
Connections:
- net +24V: now also Cf_inpflt1.1, Lf_inpflt1.1
- net +5V: now also Cff1.2, Cldo1.1, Cout1.1, Cout2.1, Rfbt1.2, U5.5 (VLDOIN), U5.8 (VOUT1), U5.9 (VOUT2)
- net GND: now also Cb_inpflt1.2, Cb_inpflt2.2, Cb_inpflt3.2, Cb_inpflt4.2, Cf_inpflt1.2, Cin2.2, Cin5.2, Cldo1.2, Cout1.2, Cout2.2, Rfbb1.1, Rt1.2, U5.11 (AGND), U5.17 (PGND), U5.18 (PGND), U5.19 (PGND), U5.20 (PGND), U5.6 (AGND)
- new net: Rt1.1, U5.12 (RT)
- new net: Cin2.1, Cin5.1, Lf_inpflt1.2, Rd_inpflt1.1, U5.1 (VIN1), U5.14 (EN), U5.16 (VIN2)
- new net: Cb_inpflt1.1, Cb_inpflt2.1, Cb_inpflt3.1, Cb_inpflt4.1, Rd_inpflt1.2
- new net: Cff1.1, Rfbb1.2, Rfbt1.1, U5.10 (FB)
- new net: U5.3 (CBOOT), U5.4 (RBOOT)
- no-connect marks 0 -> 3
Other:
- note added: "+24 to +5V converter"
- note removed: "+24V to +5V converter"
- moved on the sheet: C14, C15, C16, C17, C18, C19, C20, L1, L2, R5, R6, R7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
