Commit message: very simple algorithm ik and first simulink try
A very simple Matbal inverse kinematics algorithm and a first simulink programm which only displays the robot

File: Software/robotarm/urdf/robot_armV2SLDASM.urdf (robot description, URDF)
Before this commit: robot robot_armV2.SLDASM, 13 links, 12 joints
Links:
- link base_link: geometry collision mesh filename=..meshes/base_link.STL; visual mesh filename=../meshes/base_link.STL
- link forearm_link: geometry collision mesh filename=../meshes/forearm_link.STL; visual mesh filename=../meshes/forearm_link.STL
- link gripper_left_drive_arm_link: geometry collision mesh filename=../meshes/gripper_left_drive_arm_link.STL; visual mesh filename=../meshes/gripper_left_drive_arm_link.STL
- link gripper_left_finger_link: geometry collision mesh filename=../meshes/gripper_left_finger_link.STL; visual mesh filename=../meshes/gripper_left_finger_link.STL
- link gripper_left_support_arm_link: geometry collision mesh filename=../meshes/gripper_left_support_arm_link.STL; visual mesh filename=../meshes/gripper_left_support_arm_link.STL
- link gripper_right_drive_arm_link: geometry collision mesh filename=../meshes/gripper_right_drive_arm_link.STL; visual mesh filename=../meshes/gripper_right_drive_arm_link.STL
- link gripper_right_finger_link: geometry collision mesh filename=../meshes/gripper_right_finger_link.STL; visual mesh filename=../meshes/gripper_right_finger_link.STL
- link gripper_right_support_arm_link: geometry collision mesh filename=../meshes/gripper_right_support_arm_link.STL; visual mesh filename=../meshes/gripper_right_support_arm_link.STL
- link gripper_turn_link: geometry collision mesh filename=../meshes/gripper_turn_link.STL; visual mesh filename=../meshes/gripper_turn_link.STL
- link shoulder_link: geometry collision mesh filename=../meshes/shoulder_link.STL; visual mesh filename=../meshes/shoulder_link.STL
- link upperarm_link: geometry collision mesh filename=../meshes/upperarm_link.STL; visual mesh filename=../meshes/upperarm_link.STL
- link wrist_tilt_link: geometry collision mesh filename=../meshes/wrist_tilt_link.STL; visual mesh filename=../meshes/wrist_tilt_link.STL
- link wrist_turn_link: geometry collision mesh filename=../meshes/wrist_turn_link.STL; visual mesh filename=../meshes/wrist_turn_link.STL
Joints:
- joint gripper_left_drive_arm_joint: limit lower=-15708 upper=15708 effort=1 velocity=1 -> lower=-1.5708 upper=1.5708 effort=1 velocity=1
- joint gripper_left_finger_joint: limit lower=-15708 upper=15708 effort=1 velocity=1 -> lower=-1.5708 upper=1.5708 effort=1 velocity=1
- joint gripper_left_support_arm_joint: limit lower=0 upper=0 effort=0 velocity=0 -> lower=0 upper=6.37 effort=0 velocity=0
- joint gripper_right_drive_arm_joint: limit lower=-15708 upper=15708 effort=1 velocity=1 -> lower=-1.5708 upper=1.5708 effort=1 velocity=1
- joint gripper_right_finger_joint: limit lower=-15708 upper=15708 effort=1 velocity=1 -> lower=-1.5708 upper=1.5708 effort=1 velocity=1
- joint gripper_right_support_arm_joint: limit lower=0 upper=0 effort=0 velocity=0 -> lower=0 upper=6.37 effort=0 velocity=0

Commit message: small changes and clean up
deleted gripper controller

File: Software/robotarm/urdf/robot_armV2SLDASM.urdf (robot description, URDF)
Before this commit: robot robot_armV2.SLDASM, 13 links, 12 joints
Links:
- removed link gripper_left_drive_arm_link
- removed link gripper_left_finger_link
- removed link gripper_left_support_arm_link
- removed link gripper_right_drive_arm_link
- removed link gripper_right_finger_link
- removed link gripper_right_support_arm_link
Joints:
- removed joint gripper_left_drive_arm_joint
- removed joint gripper_left_finger_joint
- removed joint gripper_left_support_arm_joint
- removed joint gripper_right_drive_arm_joint
- removed joint gripper_right_finger_joint
- removed joint gripper_right_support_arm_joint
