File: Electrical/test_board/test_board/_autosave-test_board.kicad_pcb (KiCad board)
At the start: 2 copper layers, 29 parts, among them J10 Conn_01x04_Socket, J11 Conn_01x06_Pin, J12 Conn_01x04_Socket, J2 Conn_01x04_Socket, J3 Conn_01x06_Pin, J4 Conn_01x04_Socket, J5 Conn_01x06_Pin, J6 Conn_01x04_Socket, J7 Conn_01x06_Pin, J8 Conn_01x04_Socket, J9 Conn_01x06_Pin

Commit message: Started PCB layout for test board
Parts:
- added DRV_1: TMC5160T_V1.0, Robot:TMC5160T_Pro_V1.0_Breakout, F.Cu at (143.8, 36.7)
- added DRV_2: TMC5160T_V1.0, Robot:TMC5160T_Pro_V1.0_Breakout, F.Cu at (143.8, 61.7)
- added DRV_3: TMC5160T_V1.0, Robot:TMC5160T_Pro_V1.0_Breakout, F.Cu at (143.8, 86.7)
- added DRV_4: TMC5160T_V1.0, Robot:TMC5160T_Pro_V1.0_Breakout, F.Cu at (143.8, 111.7)
- added DRV_5: TMC5160T_V1.0, Robot:TMC5160T_Pro_V1.0_Breakout, F.Cu at (143.8, 136.7)
- added DRV_6: TMC5160T_V1.0, Robot:TMC5160T_Pro_V1.0_Breakout, F.Cu at (143.8, 161.7)
- added J1: Conn_01x06_Pin, Connector_PinHeader_2.54mm:PinHeader_1x06_P2.54mm_Vertical, F.Cu at (123.5, 32.9)
- moved J11 111.3 mm to (123.5, 157.9)
- moved J9 87.2 mm to (123.5, 132.9)
- moved J12 86.9 mm to (163.5, 158.0), turned to -90 degrees
- moved J10 77.5 mm to (163.5, 133.0), turned to -90 degrees
- moved J2 75.8 mm to (163.5, 33.0), turned to -90 degrees
- moved J8 71.1 mm to (163.5, 108.0), turned to -90 degrees
- moved J4 70.2 mm to (163.5, 58.0), turned to -90 degrees
- moved J6 68.5 mm to (163.5, 83.0), turned to -90 degrees
- moved J7 64.1 mm to (123.5, 107.9)
- moved J5 43.7 mm to (123.5, 82.9)
- moved C10 32.9 mm to (52.0, 55.5)
- moved C11 32.9 mm to (52.0, 65.0)
- moved C12 32.9 mm to (52.0, 74.6)
- moved C4 32.9 mm to (42.3, 55.5)
- moved C5 32.9 mm to (42.3, 65.0)
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