File: Electrical/test_board/test_board/_autosave-test_board.kicad_pcb (KiCad board)
At the start: 2 copper layers, 61 x 171.5 mm, 31 parts, among them J1 Conn_01x06_Pin, J10 Conn_01x04_Socket, J11 Conn_01x06_Pin, J12 Conn_01x04_Socket, J13 Screw_Terminal_01x04, J2 Conn_01x04_Socket, J3 Conn_01x06_Pin, J4 Conn_01x04_Socket, J5 Conn_01x06_Pin, J6 Conn_01x04_Socket, J7 Conn_01x06_Pin, J8 Conn_01x04_Socket, J9 Conn_01x06_Pin

Commit message: Finished testboard
Parts:
- moved J4 5.90 mm to (136.0, 70.3)
- moved J2 5.88 mm to (136.0, 45.2)
- moved J1 5.86 mm to (110.0, 45.2)
- moved J11 5.86 mm to (110.0, 170.2)
- moved J3 5.86 mm to (110.0, 70.2)
- moved J5 5.86 mm to (110.0, 95.2)
- moved J7 5.86 mm to (110.0, 120.2)
- moved J9 5.86 mm to (110.0, 145.2)
- moved J8 5.41 mm to (136.5, 120.5)
- moved J6 5.40 mm to (136.5, 95.2)
- moved J10 5.40 mm to (136.5, 145.3)
- moved J12 5.40 mm to (136.5, 170.3)
Routing:
- net Net-(DRV_2-Pin_6): track 13.5 -> 7.63 mm
- net Net-(DRV_2-Pin_10): track 13.5 -> 7.60 mm
- net Net-(DRV_2-Pin_12): track 13.5 -> 7.62 mm
- net Net-(DRV_2-Pin_8): track 13.5 -> 7.62 mm
- net Net-(DRV_1-Pin_6): track 13.5 -> 7.67 mm
- net Net-(DRV_1-Pin_12): track 13.5 -> 7.65 mm
- net Net-(DRV_1-Pin_10): track 13.5 -> 7.64 mm
- net Net-(DRV_1-Pin_8): track 13.5 -> 7.65 mm
- net Net-(DRV_6-Pin_13): track 11.8 -> 5.97 mm
- net Net-(DRV_4-Pin_15): track 11.8 -> 5.97 mm
- net Net-(DRV_1-Pin_9): track 12.8 -> 6.94 mm
- net Net-(DRV_1-Pin_7): track 12.8 -> 6.94 mm
- net Net-(DRV_1-Pin_5): track 12.8 -> 6.94 mm
- net Net-(DRV_1-Pin_3): track 12.8 -> 6.94 mm
- net Net-(DRV_6-Pin_9): track 12.8 -> 6.94 mm
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Other:
- board text added: "github.com/EmanuelKaefer/Open-robot-arm"

Commit message: Cleaned up test board
Parts:
- renumbered C13 to C10, C14 to C11, C15 to C12, C10 to C7, C11 to C8, C12 to C9, J13 to J1, J9 to J10, J10 to J11, J11 to J12, J12 to J13, J1 to J2, J2 to J3, J3 to J4, J4 to J5, J5 to J6, J6 to J7, J7 to J8, J8 to J9
Changed lines of the file:
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@@
 	)
 	(paper "A4")
+	(title_block
+		(title "Test board")
+		(date "2026-05-18")
+		(company "github.com/EmanuelKaefer/Open-robot-arm")
+	)
 	(layers
 		(0 "F.Cu" signal)
@@
 		(descr "Through hole straight pin header, 1x06, 2.54mm pitch, single row")
 		(tags "Through hole pin header THT 1x06 2.54mm single row")
-		(property "Reference" "J1"
+		(property "Reference" "J2"
 			(at 0 -2.38 0)
 			(layer "F.SilkS")
@@
 		(descr "CP, Radial series, Radial, pin pitch=2.50mm, diameter=8mm, height=10mm, Electrolytic Capacitor")
 		(tags "CP Radial series Radial pin pitch 2.50mm diameter 8mm height 10mm Electrolytic Capacitor")
-		(property "Reference" "C11"
+		(property "Reference" "C8"
 			(at 1.25 -5.25 0)
 			(layer "F.SilkS")
@@
 		(descr "Through hole straight pin header, 1x06, 2.54mm pitch, single row")
 		(tags "Through hole pin header THT 1x06 2.54mm single row")
-		(property "Reference" "J7"
+		(property "Reference" "J8"
 			(at 0 -2.38 0)
 			(layer "F.SilkS")
@@
 		(descr "JST XH series connector, B4B-XH-A (http://www.jst-mfg.com/product/pdf/eng/eXH.pdf), generated with kicad-footprint-generator")
 		(tags "connector JST XH vertical")
-		(property "Reference" "J4"
+		(property "Reference" "J5"
 			(at 3.75 -3.55 90)
 			(layer "F.SilkS")
@@
 		(descr "JST XH series connector, B4B-XH-A (http://www.jst-mfg.com/product/pdf/eng/eXH.pdf), generated with kicad-footprint-generator")
 		(tags "connector JST XH vertical")
-		(property "Reference" "J8"
+		(property "Reference" "J9"
 			(at 3.75 -3.55 90)
 			(layer "F.SilkS")
@@
 		(descr "CP, Radial series, Radial, pin pitch=2.50mm, diameter=8mm, height=10mm, Electrolytic Capacitor")
 		(tags "CP Radial series Radial pin pitch 2.50mm diameter 8mm height 10mm Electrolytic Capacitor")
-		(property "Reference" "C15"
+		(property "Reference" "C12"
 			(at 1.25 -5.25 0)
 			(layer "F.SilkS")
@@
 		(descr "Through hole straight pin header, 1x06, 2.54mm pitch, single row")
 		(tags "Through hole pin header THT 1x06 2.54mm single row")
-		(property "Reference" "J11"
+		(property "Reference" "J12"
 			(at 0 -2.38 0)
 			(layer "F.SilkS")
@@
 		(descr "JST XH series connector, B4B-XH-A (http://www.jst-mfg.com/product/pdf/eng/eXH.pdf), generated with kicad-footprint-generator")
 		(tags "connector JST XH vertical")
-		(property "Reference" "J12"
+		(property "Reference" "J13"
 			(at 3.75 -3.55 90)
 			(layer "F.SilkS")
@@
 		(descr "Terminal Block Phoenix MKDS-1,5-4-5.08, 4 pins, pitch 5.08mm, size 20.3x9.8mm, drill diameter 1.3mm, pad diameter 2.6mm, http://www.farnell.com/datasheets/100425.pdf, script-generated using https://gitlab.com/kicad/libraries/kicad-footprint-generator/-/tree/master/scripts/TerminalBlock_Phoenix")
 		(tags "THT Terminal Block Phoenix MKDS-1,5-4-5.08 pitch 5.08mm size 20.3x9.8mm drill 1.3mm pad 2.6mm")
-		(property "Reference" "J13"
+		(property "Reference" "J1"
 			(at 7.62 -6.32 0)
 			(layer "F.SilkS")
@@
 		(descr "JST XH series connector, B4B-XH-A (http://www.jst-mfg.com/product/pdf/eng/eXH.pdf), generated with kicad-footprint-generator")
 		(tags "connector JST XH vertical")
-		(property "Reference" "J2"
+		(property "Reference" "J3"
 			(at 3.75 -3.55 90)
 			(layer "F.SilkS")
@@
 		(descr "CP, Radial series, Radial, pin pitch=2.50mm, diameter=8mm, height=10mm, Electrolytic Capacitor")
 		(tags "CP Radial series Radial pin pitch 2.50mm diameter 8mm height 10mm Electrolytic Capacitor")
-		(property "Reference" "C10"
+		(property "Reference" "C7"
 			(at 1.25 -5.25 0)
 			(layer "F.SilkS")
@@
 		(descr "CP, Radial series, Radial, pin pitch=2.50mm, diameter=8mm, height=10mm, Electrolytic Capacitor")
 		(tags "CP Radial series Radial pin pitch 2.50mm diameter 8mm height 10mm Electrolytic Capacitor")
-		(property "Reference" "C14"
+		(property "Reference" "C11"
 			(at 1.25 -5.25 0)
 			(layer "F.SilkS")
@@
 		(descr "JST XH series connector, B4B-XH-A (http://www.jst-mfg.com/product/pdf/eng/eXH.pdf), generated with kicad-footprint-generator")
 		(tags "connector JST XH vertical")
-		(property "Reference" "J6"
+		(property "Reference" "J7"
 			(at 3.75 -3.55 90)
 			(layer "F.SilkS")
@@
 		(descr "CP, Radial series, Radial, pin pitch=2.50mm, diameter=8mm, height=10mm, Electrolytic Capacitor")
 		(tags "CP Radial series Radial pin pitch 2.50mm diameter 8mm height 10mm Electrolytic Capacitor")
-		(property "Reference" "C12"
+		(property "Reference" "C9"
 			(at 1.25 -5.25 0)
 			(layer "F.SilkS")
@@
 		(descr "CP, Radial series, Radial, pin pitch=2.50mm, diameter=8mm, height=10mm, Electrolytic Capacitor")
 		(tags "CP Radial series Radial pin pitch 2.50mm diameter 8mm height 10mm Electrolytic Capacitor")
-		(property "Reference" "C13"
+		(property "Reference" "C10"
 			(at 1.25 -5.25 0)
 			(layer "F.SilkS")
@@
 		(descr "Through hole straight pin header, 1x06, 2.54mm pitch, single row")
 		(tags "Through hole pin header THT 1x06 2.54mm single row")
-		(property "Reference" "J5"
+		(property "Reference" "J6"
 			(at 0 -2.38 0)
 			(layer "F.SilkS")
@@
 		(descr "Through hole straight pin header, 1x06, 2.54mm pitch, single row")
 		(tags "Through hole pin header THT 1x06 2.54mm single row")
-		(property "Reference" "J3"
+		(property "Reference" "J4"
 			(at 0 -2.38 0)
 			(layer "F.SilkS")
@@
 		(descr "Through hole straight pin header, 1x06, 2.54mm pitch, single row")
 		(tags "Through hole pin header THT 1x06 2.54mm single row")
-		(property "Reference" "J9"
+		(property "Reference" "J10"
 			(at 0 -2.38 0)
 			(layer "F.SilkS")
@@
 		(descr "JST XH series connector, B4B-XH-A (http://www.jst-mfg.com/product/pdf/eng/eXH.pdf), generated with kicad-footprint-generator")
 		(tags "connector JST XH vertical")
-		(property "Reference" "J10"
+		(property "Reference" "J11"
 			(at 3.75 -3.55 90)
 			(layer "F.SilkS")
