File: Electrical/test_board/test_board/test_board.kicad_pcb (KiCad board)
At the start: 2 copper layers, 31 parts, among them J1 Conn_01x06_Pin, J10 Conn_01x04_Socket, J11 Conn_01x06_Pin, J12 Conn_01x04_Socket, J13 Screw_Terminal_01x04, J2 Conn_01x04_Socket, J3 Conn_01x06_Pin, J4 Conn_01x04_Socket, J5 Conn_01x06_Pin, J6 Conn_01x04_Socket, J7 Conn_01x06_Pin, J8 Conn_01x04_Socket, J9 Conn_01x06_Pin

Commit message: Updated testboard
Parts:
- moved J13 13.0 mm to (137.2, 27.9)
- moved J1 11.1 mm to (104.1, 45.2)
- moved J3 11.1 mm to (104.1, 70.2)
- moved J5 11.1 mm to (104.1, 95.2)
- moved J11 11.1 mm to (104.1, 170.2)
- moved J7 11.1 mm to (104.1, 120.2)
- moved J9 11.1 mm to (104.1, 145.2)
- moved DRV_4 9.73 mm to (122.2, 124.0)
- moved C1 9.73 mm to (152.4, 40.3)
- moved C11 9.73 mm to (152.4, 140.4)
- moved C12 9.73 mm to (152.4, 165.4)
- moved C13 9.73 mm to (152.4, 123.9)
- moved C14 9.73 mm to (152.4, 148.9)
- moved C15 9.73 mm to (152.4, 173.9)
- moved C5 9.73 mm to (152.4, 73.9)
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Routing:
- net GND: track 521.8 -> 0.00 mm
- net +3.3V: track 335.9 -> 175.6 mm
- net Net-(DRV_5-Pin_15): track 14.0 -> 11.8 mm
- net Net-(DRV_6-Pin_7): track 15.0 -> 12.8 mm
- net Net-(DRV_6-Pin_5): track 15.0 -> 12.8 mm
- net Net-(DRV_5-Pin_7): track 15.0 -> 12.8 mm
- net Net-(DRV_5-Pin_5): track 15.0 -> 12.8 mm
- net Net-(DRV_4-Pin_9): track 15.0 -> 12.8 mm
- net Net-(DRV_4-Pin_5): track 15.0 -> 12.8 mm
- net Net-(DRV_3-Pin_9): track 15.0 -> 12.8 mm
- net Net-(DRV_3-Pin_5): track 15.0 -> 12.8 mm
- net Net-(DRV_2-Pin_9): track 15.0 -> 12.8 mm
- net Net-(DRV_2-Pin_5): track 15.0 -> 12.8 mm
- net Net-(DRV_1-Pin_9): track 15.0 -> 12.8 mm
- net Net-(DRV_1-Pin_7): track 15.0 -> 12.8 mm
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Other:
- board outline added: 61 x 170.2 mm

Commit message: Finished testboard
Parts:
- moved J4 5.90 mm to (136.0, 70.3)
- moved J2 5.88 mm to (136.0, 45.2)
- moved J1 5.86 mm to (110.0, 45.2)
- moved J11 5.86 mm to (110.0, 170.2)
- moved J3 5.86 mm to (110.0, 70.2)
- moved J5 5.86 mm to (110.0, 95.2)
- moved J7 5.86 mm to (110.0, 120.2)
- moved J9 5.86 mm to (110.0, 145.2)
- moved J8 5.41 mm to (136.5, 120.5)
- moved J6 5.40 mm to (136.5, 95.2)
- moved J10 5.40 mm to (136.5, 145.3)
- moved J12 5.40 mm to (136.5, 170.3)
- moved C11 1.61 mm to (154.0, 140.6)
- moved C12 1.61 mm to (154.0, 165.6)
- moved C13 1.61 mm to (154.0, 124.1)
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Connections:
- J13 pad 1: +3.3V -> +24V
- J13 pad 2: +24V -> GND
- J13 pad 3: GND -> +3.3V
Routing:
- net +24V: track 294.7 -> 319.3 mm
- net Net-(DRV_2-Pin_6): track 13.5 -> 7.63 mm
- net Net-(DRV_2-Pin_10): track 13.5 -> 7.60 mm
- net Net-(DRV_2-Pin_12): track 13.5 -> 7.62 mm
- net Net-(DRV_2-Pin_8): track 13.5 -> 7.62 mm
- net Net-(DRV_1-Pin_6): track 13.5 -> 7.67 mm
- net Net-(DRV_1-Pin_12): track 13.5 -> 7.65 mm
- net Net-(DRV_1-Pin_10): track 13.5 -> 7.64 mm
- net Net-(DRV_1-Pin_8): track 13.5 -> 7.65 mm
- net Net-(DRV_6-Pin_13): track 11.8 -> 5.97 mm
- net Net-(DRV_4-Pin_15): track 11.8 -> 5.97 mm
- net Net-(DRV_1-Pin_9): track 12.8 -> 6.94 mm
- net Net-(DRV_1-Pin_7): track 12.8 -> 6.94 mm
- net Net-(DRV_1-Pin_5): track 12.8 -> 6.94 mm
- net Net-(DRV_1-Pin_3): track 12.8 -> 6.94 mm
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- added copper zone on B.Cu, net GND
Other:
- board size 61 x 170.2 mm -> 61 x 171.5 mm

Commit message: Adjusted test board
Parts:
- moved C3 91.4 mm to (145.0, 181.5), turned to 180 degrees
- moved C12 78.1 mm to (145.0, 96.5), turned to 180 degrees
- moved C6 72.9 mm to (145.0, 171.5), turned to 180 degrees
- moved C9 59.8 mm to (145.0, 106.5), turned to 180 degrees
- moved C7 42.0 mm to (145.0, 156.5), turned to 180 degrees
- moved C11 29.0 mm to (145.0, 121.5), turned to 180 degrees
- moved C10 24.1 mm to (145.0, 146.5), turned to 180 degrees
- moved C8 12.8 mm to (145.0, 131.5), turned to 180 degrees
- moved C4 11.6 mm to (145.0, 56.5), turned to 180 degrees
- moved C5 11.6 mm to (145.0, 81.5), turned to 180 degrees
- moved C2 10.8 mm to (145.0, 71.5), turned to 180 degrees
- moved C1 10.8 mm to (145.0, 46.5), turned to 180 degrees
- renumbered C13 to C10, C14 to C11, C15 to C12, C10 to C7, C11 to C8, C12 to C9, J13 to J1, J9 to J10, J10 to J11, J11 to J12, J12 to J13, J1 to J2, J2 to J3, J3 to J4, J4 to J5, J5 to J6, J6 to J7, J7 to J8, J8 to J9
Routing:
- net +24V: track 319.3 -> 326.3 mm
Other:
- board text added: "github.com/EmanuelKaefer/Open-robot-arm"

Commit message: Last changes before first milling to Test board
Parts:
- added D1: D_TVS, Diode_THT:D_DO-201AD_P15.24mm_Horizontal, F.Cu at (149.9, 38.6)
- moved C10 3.39 mm to (144.8, 149.9)
- moved C11 3.39 mm to (144.8, 124.9)
- moved C12 3.39 mm to (144.8, 99.9)
- moved C2 3.39 mm to (144.8, 74.9)
- moved C3 3.39 mm to (144.8, 184.9)
- moved C5 3.39 mm to (144.8, 84.9)
- moved C6 3.39 mm to (144.8, 174.9)
- moved C7 3.39 mm to (144.8, 159.9)
- moved C8 3.39 mm to (144.8, 134.9)
- moved C9 3.39 mm to (144.8, 109.9)
- moved J11 3.39 mm to (136.3, 148.7)
- moved J13 3.39 mm to (136.3, 173.7)
- moved J7 3.39 mm to (136.3, 98.6)
- moved J9 3.39 mm to (136.3, 123.9)
- moved DRV_2 3.39 mm to (121.9, 77.4)
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Other:
- board size 61 x 171.5 mm -> 61 x 176.5 mm

Commit message: improvement
Other:
- board text added: "github.com/EmanuelKaefer/Open-robot-arm CERN-OHL-S-2.0"
- board text removed: "github.com/EmanuelKaefer/Open-robot-arm"
Changed lines of the file:
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@@
 		(tenting front back)
 		(pcbplotparams
-			(layerselection 0x00000000_00000000_55555555_5755f5ff)
+			(layerselection 0x00000000_00000000_55555555_575555d4)
 			(plot_on_all_layers_selection 0x00000000_00000000_00000000_00000000)
 			(disableapertmacros no)
@@
 			(outputformat 1)
 			(mirror no)
-			(drillshape 1)
+			(drillshape 0)
 			(scaleselection 1)
 			(outputdirectory "")
@@
 		(layer "Edge.Cuts")
 	)
-	(gr_text "github.com/EmanuelKaefer/Open-robot-arm"
-		(at 146.259 22.376844 0)
-		(layer "B.SilkS")
-		(effects
-			(font
-				(size 1 1)
-				(thickness 0.125)
-			)
-			(justify left bottom mirror)
-		)
-	)
 	(gr_text ""
 		(at 5 5 0)
@@
 		)
 	)
+	(gr_text "github.com/EmanuelKaefer/Open-robot-arm\nCERN-OHL-S-2.0"
+		(at 100.5 109.5 270)
+		(layer "User.1")
+		(effects
+			(font
+				(size 1.5 1.5)
+				(thickness 0.3)
+				(bold yes)
+			)
+			(justify bottom)
+		)
+	)
