File: Electrical/test_board/test_board/test_board.kicad_pcb (KiCad board)
At the start: 2 copper layers, 61 x 176.5 mm, 32 parts, among them J1 Screw_Terminal_01x04, J10 Conn_01x06_Pin, J11 Conn_01x04_Socket, J12 Conn_01x06_Pin, J13 Conn_01x04_Socket, J2 Conn_01x06_Pin, J3 Conn_01x04_Socket, J4 Conn_01x06_Pin, J5 Conn_01x04_Socket, J6 Conn_01x06_Pin, J7 Conn_01x04_Socket, J8 Conn_01x06_Pin, J9 Conn_01x04_Socket

Commit message: Fixed the whole test thing
Parts:
- removed the J2 at (109.8, 48.6)
- removed the J4 at (109.8, 73.6)
- removed the J6 at (109.8, 98.6)
- added J1: Conn_01x03_Pin, Connector_PinHeader_2.54mm:PinHeader_1x03_P2.54mm_Vertical, F.Cu at (109.7, 31.5)
- added J14: Conn_01x03_Pin, Connector_PinHeader_2.54mm:PinHeader_1x03_P2.54mm_Vertical, F.Cu at (109.7, 127.3)
- added J6: Conn_01x03_Pin, Connector_PinHeader_2.54mm:PinHeader_1x03_P2.54mm_Vertical, F.Cu at (109.7, 52.4)
- added J6: Conn_01x03_Pin, Connector_PinHeader_2.54mm:PinHeader_1x03_P2.54mm_Vertical, F.Cu at (109.7, 77.4)
- added R1: 0Ohm, Resistor_THT:R_Axial_DIN0207_L6.3mm_D2.5mm_P10.16mm_Horizontal, F.Cu at (101.9, 45.0)
- added R10: 0Ohm, Resistor_THT:R_Axial_DIN0207_L6.3mm_D2.5mm_P10.16mm_Horizontal, F.Cu at (101.9, 123.0)
- added R11: 0Ohm, Resistor_THT:R_Axial_DIN0207_L6.3mm_D2.5mm_P10.16mm_Horizontal, F.Cu at (101.9, 148.0)
- added R12: 0Ohm, Resistor_THT:R_Axial_DIN0207_L6.3mm_D2.5mm_P10.16mm_Horizontal, F.Cu at (101.9, 173.0)
- added R2: 0Ohm, Resistor_THT:R_Axial_DIN0207_L6.3mm_D2.5mm_P10.16mm_Horizontal, F.Cu at (101.9, 70.0)
- added R3: 0Ohm, Resistor_THT:R_Axial_DIN0207_L6.3mm_D2.5mm_P10.16mm_Horizontal, F.Cu at (101.9, 95.0)
- added R4: 0Ohm, Resistor_THT:R_Axial_DIN0207_L6.3mm_D2.5mm_P10.16mm_Horizontal, F.Cu at (101.9, 48.0)
- added R5: 0Ohm, Resistor_THT:R_Axial_DIN0207_L6.3mm_D2.5mm_P10.16mm_Horizontal, F.Cu at (101.9, 73.0)
- added R6: 0Ohm, Resistor_THT:R_Axial_DIN0207_L6.3mm_D2.5mm_P10.16mm_Horizontal, F.Cu at (101.9, 98.0)
- added R7: 0Ohm, Resistor_THT:R_Axial_DIN0207_L6.3mm_D2.5mm_P10.16mm_Horizontal, F.Cu at (101.9, 120.0)
- added R8: 0Ohm, Resistor_THT:R_Axial_DIN0207_L6.3mm_D2.5mm_P10.16mm_Horizontal, F.Cu at (101.9, 145.0)
- added R9: 0Ohm, Resistor_THT:R_Axial_DIN0207_L6.3mm_D2.5mm_P10.16mm_Horizontal, F.Cu at (101.9, 170.0)
- J10, J12, J8: value Conn_01x06_Pin -> Conn_01x03_Pin; footprint Connector_PinHeader_2.54mm:PinHeader_1x06_P2.54mm_Vertical -> Connector_PinHeader_2.54mm:PinHeader_1x03_P2.54mm_Vertical
- moved J10 28.8 mm to (109.7, 177.4)
- moved J8 21.2 mm to (109.7, 102.3)
- moved J12 21.2 mm to (109.2, 152.4)
- moved J2 1.35 mm to (136.1, 30.2)
- moved DRV_2 1.35 mm to (121.1, 76.3)
- moved DRV_3 1.35 mm to (121.1, 101.3)
- moved DRV_4 1.35 mm to (121.1, 126.3)
- moved DRV_1 1.35 mm to (121.1, 51.3)
- moved C10 1.35 mm to (144.0, 148.8)
- moved C11 1.35 mm to (144.0, 123.8)
- moved C12 1.35 mm to (144.0, 98.8)
- moved C2 1.35 mm to (144.0, 73.8)
- moved C3 1.35 mm to (144.0, 183.8)
- moved C5 1.35 mm to (144.0, 83.8)
- moved C6 1.35 mm to (144.0, 173.8)
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- renumbered J11 to J10, J13 to J11, J1 to J2, J5 to J4, J7 to J5
Connections:
- DRV_1 pad 9: Net-(DRV_1-Pin_9) -> MISO
- DRV_2 pad 9: Net-(DRV_2-Pin_9) -> MISO
- DRV_3 pad 9: Net-(DRV_3-Pin_9) -> MISO
- DRV_4 pad 9: Net-(DRV_4-Pin_9) -> MISO
- DRV_5 pad 9: Net-(DRV_5-Pin_9) -> MISO
- DRV_6 pad 9: Net-(DRV_6-Pin_9) -> MISO
- J10 pad 1: Net-(DRV_5-Pin_3) -> Net-(DRV_6-Pin_7)
- J10 pad 2: Net-(DRV_5-Pin_5) -> Net-(DRV_6-Pin_13)
- J10 pad 3: Net-(DRV_5-Pin_7) -> Net-(DRV_6-Pin_15)
- J12 pad 1: Net-(DRV_6-Pin_3) -> Net-(DRV_5-Pin_7)
- J12 pad 2: Net-(DRV_6-Pin_5) -> Net-(DRV_5-Pin_13)
- J12 pad 3: Net-(DRV_6-Pin_7) -> Net-(DRV_5-Pin_15)
- J8 pad 1: Net-(DRV_4-Pin_3) -> Net-(DRV_3-Pin_7)
- J8 pad 2: Net-(DRV_4-Pin_5) -> Net-(DRV_3-Pin_13)
- J8 pad 3: Net-(DRV_4-Pin_7) -> Net-(DRV_3-Pin_15)
Routing:
- net MISO: track 0.00 -> 157.7 mm
- net SCK: track 0.00 -> 156.9 mm
- net MOSI: track 0.00 -> 156.4 mm
- net Net-(DRV_3-Pin_9): track 6.94 -> 0.00 mm
- net Net-(DRV_2-Pin_9): track 6.94 -> 0.00 mm
- net Net-(DRV_1-Pin_9): track 6.94 -> 0.00 mm
- net Net-(DRV_6-Pin_9): track 6.94 -> 0.00 mm
- net Net-(DRV_5-Pin_9): track 6.94 -> 0.00 mm
- net Net-(DRV_5-Pin_5): track 6.94 -> 0.00 mm
- net Net-(DRV_4-Pin_9): track 6.94 -> 0.00 mm
- net Net-(DRV_5-Pin_3): track 6.94 -> 0.08 mm
- net Net-(DRV_6-Pin_3): track 6.94 -> 2.81 mm
- net Net-(DRV_1-Pin_3): track 6.94 -> 2.81 mm
- net Net-(DRV_4-Pin_3): track 6.94 -> 2.81 mm
- net Net-(DRV_3-Pin_3): track 6.94 -> 2.81 mm
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Other:
- board size 61 x 176.5 mm -> 57.5 x 175 mm

Commit message: Final adjustments to test board (hopefully)
Routing:
- net +3.3V: track 171.4 -> 183.2 mm
- net +24V: track 326.3 -> 331.1 mm
Other:
- board size 57.5 x 175 mm -> 57.5 x 176 mm
Changed lines of the file:
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@@
 	)
 	(gr_line
-		(start 155 190)
-		(end 107 190)
+		(start 155 191)
+		(end 107 191)
 		(stroke
 			(width 0.05)
@@
 	)
 	(gr_line
-		(start 107 190)
-		(end 100 190)
+		(start 107 191)
+		(end 100 191)
 		(stroke
 			(width 0.05)
@@
 	)
 	(gr_line
-		(start 100 190)
-		(end 97.5 190)
+		(start 100 191)
+		(end 97.5 191)
 		(stroke
 			(width 0.05)
@@
 	)
 	(gr_line
-		(start 155 190)
+		(start 155 191)
 		(end 155 22.5)
 		(stroke
@@
 	(gr_line
 		(start 97.5 22.5)
-		(end 97.5 190)
+		(end 97.5 191)
 		(stroke
 			(width 0.05)
@@
 	)
 	(gr_text "github.com/EmanuelKaefer/Open-robot-arm\nCERN-OHL-S-2.0"
-		(at 78.5 105 270)
+		(at 126.5 19 0)
 		(layer "User.1")
 		(effects
 			(font
-				(size 1.5 1.5)
-				(thickness 0.3)
+				(size 1 1)
+				(thickness 0.2)
 				(bold yes)
 			)
@@
 	)
 	(segment
-		(start 148.47 92.563156)
-		(end 127.531 92.563156)
-		(width 2.5)
-		(layer "B.Cu")
-		(net 1)
-	)
-	(segment
 		(start 148.97 93.063156)
 		(end 148.97 116.903156)
@@
 	)
 	(segment
+		(start 127.371 142.403156)
+		(end 128.274156 141.5)
+		(width 2.5)
+		(layer "B.Cu")
+		(net 1)
+	)
+	(segment
 		(start 145.849 107.776844)
 		(end 145.569 107.496844)
@@
 	)
 	(segment
+		(start 148.47 67.563156)
+		(end 147.406844 66.5)
+		(width 2.5)
+		(layer "B.Cu")
+		(net 1)
+	)
+	(segment
 		(start 151.211 42.403156)
 		(end 151.371 42.563156)
 		(width 0.2)
+		(layer "B.Cu")
+		(net 1)
+	)
+	(segment
+		(start 148.47 92.563156)
+		(end 147.406844 91.5)
+		(width 2.5)
 		(layer "B.Cu")
 		(net 1)
@@
 	)
 	(segment
+		(start 147.566844 41.5)
+		(end 148.47 42.403156)
+		(width 2.5)
+		(layer "B.Cu")
+		(net 1)
+	)
+	(segment
 		(start 148.97 92.063156)
 		(end 148.47 92.563156)
@@
 	)
 	(segment
+		(start 128.274156 116.5)
+		(end 147.566844 116.5)
+		(width 2.5)
+		(layer "B.Cu")
+		(net 1)
+	)
+	(segment
 		(start 127.531 92.563156)
 		(end 127.371 92.403156)
@@
 	)
 	(segment
-		(start 127.371 117.403156)
-		(end 148.47 117.403156)
+		(start 128.274156 141.5)
+		(end 147.566844 141.5)
+		(width 2.5)
+		(layer "B.Cu")
+		(net 1)
+	)
+	(segment
+		(start 127.371 42.403156)
+		(end 128.274156 41.5)
+		(width 2.5)
+		(layer "B.Cu")
+		(net 1)
+	)
+	(segment
+		(start 147.406844 91.5)
+		(end 128.594156 91.5)
 		(width 2.5)
 		(layer "B.Cu")
@@
 	)
 	(segment
+		(start 127.371 117.403156)
+		(end 128.274156 116.5)
+		(width 2.5)
+		(layer "B.Cu")
+		(net 1)
+	)
+	(segment
 		(start 148.47 142.403156)
 		(end 148.97 142.903156)
@@
 	)
 	(segment
-		(start 127.371 167.403156)
-		(end 147.97 167.403156)
+		(start 128.594156 91.5)
+		(end 127.531 92.563156)
+		(width 2.5)
+		(layer "B.Cu")
+		(net 1)
+	)
+	(segment
+		(start 128.274156 166.5)
+		(end 147.066844 166.5)
 		(width 2.5)
 		(layer "B.Cu")
@@
 	)
 	(segment
+		(start 147.066844 166.5)
+		(end 147.97 167.403156)
+		(width 2.5)
+		(layer "B.Cu")
+		(net 1)
+	)
+	(segment
 		(start 145.569 107.496844)
 		(end 145.57 107.497844)
@@
 		(start 151.371 67.563156)
 		(end 148.47 67.563156)
+		(width 2.5)
+		(layer "B.Cu")
+		(net 1)
+	)
+	(segment
+		(start 147.566844 116.5)
+		(end 148.47 117.403156)
+		(width 2.5)
+		(layer "B.Cu")
+		(net 1)
+	)
+	(segment
+		(start 127.371 167.403156)
+		(end 128.274156 166.5)
+		(width 2.5)
+		(layer "B.Cu")
+		(net 1)
+	)
+	(segment
+		(start 147.566844 141.5)
+		(end 148.47 142.403156)
 		(width 2.5)
 		(layer "B.Cu")
@@
 	)
 	(segment
-		(start 148.47 67.563156)
-		(end 127.531 67.563156)
+		(start 128.274156 41.5)
+		(end 147.566844 41.5)
 		(width 2.5)
 		(layer "B.Cu")
@@
 	)
 	(segment
-		(start 127.371 142.403156)
-		(end 148.47 142.403156)
+		(start 128.594156 66.5)
+		(end 127.531 67.563156)
 		(width 2.5)
 		(layer "B.Cu")
@@
 	)
 	(segment
-		(start 127.371 42.403156)
-		(end 148.47 42.403156)
-		(width 2.5)
-		(layer "B.Cu")
-		(net 1)
-	)
-	(segment
-		(start 123.43 161.584156)
-		(end 123.43 178.702156)
-		(width 0.5)
-		(layer "B.Cu")
-		(net 3)
-	)
-	(segment
-		(start 127.371 132.643156)
-		(end 123.43 136.584156)
-		(width 0.5)
-		(layer "B.Cu")
-		(net 3)
+		(start 147.406844 66.5)
+		(end 128.594156 66.5)
+		(width 2.5)
+		(layer "B.Cu")
+		(net 1)
 	)
 	(segment
@@
 	)
 	(segment
-		(start 123.43 61.584156)
+		(start 123.43 153.5)
+		(end 123.43 153.702156)
+		(width 0.5)
+		(layer "B.Cu")
+		(net 3)
+	)
+	(segment
+		(start 123.43 78.702156)
+		(end 123.43 103.702156)
+		(width 0.5)
+		(layer "B.Cu")
+		(net 3)
+	)
+	(segment
+		(start 123.43 103.702156)
+		(end 123.43 128.702156)
+		(width 0.5)
+		(layer "B.Cu")
+		(net 3)
+	)
+	(segment
+		(start 123.43 78.702156)
+		(end 127.371 82.643156)
+		(width 0.5)
+		(layer "B.Cu")
+		(net 3)
+	)
+	(segment
+		(start 123.43 103.702156)
+		(end 127.371 107.643156)
+		(width 0.5)
+		(layer "B.Cu")
+		(net 3)
+	)
+	(segment
+		(start 123.43 153.5)
+		(end 123.43 178.702156)
+		(width 0.5)
+		(layer "B.Cu")
+		(net 3)
+	)
+	(segment
+		(start 123.43 53.702156)
 		(end 123.43 78.702156)
+		(width 0.5)
+		(layer "B.Cu")
+		(net 3)
+	)
+	(segment
+		(start 123.43 53.702156)
+		(end 123.43 32.76)
+		(width 0.5)
+		(layer "B.Cu")
+		(net 3)
+	)
+	(segment
+		(start 123.43 128.702156)
+		(end 123.43 153.5)
+		(width 0.5)
+		(layer "B.Cu")
+		(net 3)
+	)
+	(segment
+		(start 123.43 178.702156)
+		(end 127.371 182.643156)
+		(width 0.5)
+		(layer "B.Cu")
+		(net 3)
+	)
+	(segment
+		(start 127.371 57.643156)
+		(end 123.43 53.702156)
+		(width 0.5)
+		(layer "B.Cu")
+		(net 3)
+	)
+	(segment
+		(start 123.43 32.76)
+		(end 125.97 30.22)
 		(width 0.5)
 		(layer "B.Cu")
@@
 	)
 	(segment
-		(start 127.371 57.643156)
-		(end 123.43 61.584156)
-		(width 0.5)
-		(layer "B.Cu")
-		(net 3)
-	)
-	(segment
-		(start 123.43 103.702156)
-		(end 127.371 107.643156)
-		(width 0.5)
-		(layer "B.Cu")
-		(net 3)
-	)
-	(segment
-		(start 123.43 53.702156)
-		(end 123.43 32.76)
-		(width 0.5)
-		(layer "B.Cu")
-		(net 3)
-	)
-	(segment
-		(start 127.371 82.643156)
-		(end 123.43 86.584156)
-		(width 0.5)
-		(layer "B.Cu")
-		(net 3)
-	)
-	(segment
-		(start 127.371 157.643156)
-		(end 123.43 161.584156)
-		(width 0.5)
-		(layer "B.Cu")
-		(net 3)
-	)
-	(segment
-		(start 123.43 111.584156)
-		(end 123.43 128.702156)
-		(width 0.5)
-		(layer "B.Cu")
-		(net 3)
-	)
-	(segment
-		(start 123.43 86.584156)
-		(end 123.43 103.702156)
-		(width 0.5)
-		(layer "B.Cu")
-		(net 3)
-	)
-	(segment
-		(start 123.43 178.702156)
-		(end 127.371 182.643156)
-		(width 0.5)
-		(layer "B.Cu")
-		(net 3)
-	)
-	(segment
-		(start 127.371 107.643156)
-		(end 123.43 111.584156)
-		(width 0.5)
-		(layer "B.Cu")
-		(net 3)
-	)
-	(segment
-		(start 127.371 57.643156)
-		(end 123.43 53.702156)
-		(width 0.5)
-		(layer "B.Cu")
-		(net 3)
-	)
-	(segment
-		(start 123.43 32.76)
-		(end 125.97 30.22)
-		(width 0.5)
-		(layer "B.Cu")
-		(net 3)
-	)
-	(segment
-		(start 123.43 136.584156)
-		(end 123.43 153.702156)
-		(width 0.5)
-		(layer "B.Cu")
-		(net 3)
-	)
-	(segment
-		(start 123.43 78.702156)
-		(end 127.371 82.643156)
-		(width 0.5)
-		(layer "B.Cu")
-		(net 3)
-	)
-	(segment
 		(start 134.995 52.53)
 		(end 127.404156 52.53)
@@
 		(layer "B.Cu")
 		(hatch edge 0.5)
-		(connect_pads
+		(connect_pads yes
 			(clearance 0.5)
 		)
@@
 		(polygon
 			(pts
-				(xy 97.5 190) (xy 155 190) (xy 155 22.5) (xy 147.5 15) (xy 105 15) (xy 97.5 22.5)
+				(xy 97.5 191) (xy 155 191) (xy 155 22.5) (xy 147.5 15) (xy 105 15) (xy 97.5 22.5)
 			)
 		)

Commit message: Optic
Parts:
- moved J2 2.05 mm to (134.1, 29.8)
Routing:
- net Net-(DRV_5-Pin_5): track 0.00 -> 3.01 mm
- net Net-(DRV_5-Pin_3): track 0.08 -> 2.81 mm
- net +24V: track 331.1 -> 332.2 mm

Commit message: Optical adjustments
Routing:
- net +3.3V: track 182.9 -> 203.3 mm
