File: Electrical/test_board/test_board/test_board.kicad_sch (KiCad schematic)
At the start: 0 parts

Commit message: Made and added footprint for tmc5160t pro v1.0
Parts:
- added C1, C10, C11, C12, C16, C17, C18, C2, C3, C7, C8, C9: 100nF, Capacitor_THT:CP_Radial_D8.0mm_P2.50mm, symbol Device:C
- added C13, C14, C15, C4, C5, C6: 100uF, Capacitor_THT:CP_Radial_D8.0mm_P2.50mm, symbol Device:C
- added DRV_1, DRV_2, DRV_3, DRV_4, DRV_5, DRV_6: TMC5160T_V1.0, PinSocket_2x08_P2.54mm, symbol Connector_Generic:Conn_02x08_Odd_Even
- added J1: Conn_01x06_Pin, symbol Connector:Conn_01x06_Pin
- added J10, J12, J2, J4, J6, J8: Conn_01x04_Socket, Connector_JST:JST_XH_B4B-XH-A_1x04_P2.50mm_Vertical, symbol Connector:Conn_01x04_Socket
- added J11, J3, J5, J7, J9: Conn_01x06_Pin, Connector_PinHeader_2.54mm:PinHeader_1x06_P2.54mm_Vertical, symbol Connector:Conn_01x06_Pin
Connections:
- new net: DRV_2.3 (Pin_3), J3.1 (Pin_1)
- new net: DRV_2.5 (Pin_5), J3.2 (Pin_2)
- new net: DRV_2.7 (Pin_7), J3.3 (Pin_3)
- new net: DRV_2.9 (Pin_9), J3.4 (Pin_4)
- new net: DRV_2.13 (Pin_13), J3.5 (Pin_5)
- new net: DRV_2.15 (Pin_15), J3.6 (Pin_6)
- new net: DRV_4.3 (Pin_3), J7.1 (Pin_1)
- new net: DRV_4.5 (Pin_5), J7.2 (Pin_2)
- new net: DRV_4.7 (Pin_7), J7.3 (Pin_3)
- new net: DRV_4.9 (Pin_9), J7.4 (Pin_4)
- new net: DRV_4.13 (Pin_13), J7.5 (Pin_5)
- new net: DRV_4.15 (Pin_15), J7.6 (Pin_6)
- new net: DRV_3.6 (Pin_6), J6.1 (Pin_1)
- new net: DRV_3.8 (Pin_8), J6.2 (Pin_2)
- new net: DRV_3.10 (Pin_10), J6.3 (Pin_3)
- new net: DRV_3.12 (Pin_12), J6.4 (Pin_4)
- new net: DRV_5.6 (Pin_6), J10.1 (Pin_1)
- new net: DRV_5.8 (Pin_8), J10.2 (Pin_2)
- new net: DRV_5.10 (Pin_10), J10.3 (Pin_3)
- new net: DRV_5.12 (Pin_12), J10.4 (Pin_4)
- new net: DRV_3.3 (Pin_3), J5.1 (Pin_1)
- new net: DRV_3.5 (Pin_5), J5.2 (Pin_2)
- new net: DRV_3.7 (Pin_7), J5.3 (Pin_3)
- new net: DRV_3.9 (Pin_9), J5.4 (Pin_4)
- new net: DRV_3.13 (Pin_13), J5.5 (Pin_5)
- new net: DRV_3.15 (Pin_15), J5.6 (Pin_6)
- new net: DRV_1.3 (Pin_3), J1.1 (Pin_1)
- new net: DRV_1.5 (Pin_5), J1.2 (Pin_2)
- new net: DRV_1.7 (Pin_7), J1.3 (Pin_3)
- new net: DRV_1.9 (Pin_9), J1.4 (Pin_4)
- new net: DRV_1.13 (Pin_13), J1.5 (Pin_5)
- new net: DRV_1.15 (Pin_15), J1.6 (Pin_6)
- new net: DRV_1.10 (Pin_10), J2.3 (Pin_3)
- new net: DRV_1.12 (Pin_12), J2.4 (Pin_4)
- new net: DRV_1.6 (Pin_6), J2.1 (Pin_1)
- new net: DRV_1.8 (Pin_8), J2.2 (Pin_2)
- new net: DRV_2.6 (Pin_6), J4.1 (Pin_1)
- new net: DRV_2.8 (Pin_8), J4.2 (Pin_2)
- new net: DRV_2.10 (Pin_10), J4.3 (Pin_3)
- new net: DRV_2.12 (Pin_12), J4.4 (Pin_4)
- new net: DRV_6.3 (Pin_3), J11.1 (Pin_1)
- new net: DRV_6.5 (Pin_5), J11.2 (Pin_2)
- new net: DRV_6.7 (Pin_7), J11.3 (Pin_3)
- new net: DRV_6.9 (Pin_9), J11.4 (Pin_4)
- new net: DRV_6.13 (Pin_13), J11.5 (Pin_5)
- new net: DRV_6.15 (Pin_15), J11.6 (Pin_6)
- new net: DRV_6.6 (Pin_6), J12.1 (Pin_1)
- new net: DRV_6.8 (Pin_8), J12.2 (Pin_2)
- new net: DRV_6.10 (Pin_10), J12.3 (Pin_3)
- new net: DRV_6.12 (Pin_12), J12.4 (Pin_4)
- new net: DRV_5.3 (Pin_3), J9.1 (Pin_1)
- new net: DRV_5.5 (Pin_5), J9.2 (Pin_2)
- new net: DRV_5.7 (Pin_7), J9.3 (Pin_3)
- new net: DRV_5.9 (Pin_9), J9.4 (Pin_4)
- new net: DRV_5.13 (Pin_13), J9.5 (Pin_5)
- new net: DRV_5.15 (Pin_15), J9.6 (Pin_6)
- new net: DRV_4.6 (Pin_6), J8.1 (Pin_1)
- new net: DRV_4.8 (Pin_8), J8.2 (Pin_2)
- new net: DRV_4.10 (Pin_10), J8.3 (Pin_3)
- new net: DRV_4.12 (Pin_12), J8.4 (Pin_4)
- new net +24V: C1.1, C10.1, C11.1, C12.1, C13.1, C14.1, C15.1, C2.1, C3.1, C4.1, C5.1, C6.1, DRV_1.2 (Pin_2), DRV_2.2 (Pin_2), DRV_3.2 (Pin_2), DRV_4.2 (Pin_2), DRV_5.2 (Pin_2), DRV_6.2 (Pin_2)
- new net +3.3V: C16.1, C17.1, C18.1, C7.1, C8.1, C9.1, DRV_1.14 (Pin_14), DRV_2.14 (Pin_14), DRV_3.14 (Pin_14), DRV_4.14 (Pin_14), DRV_5.14 (Pin_14), DRV_6.14 (Pin_14)
- new net GND: C1.2, C10.2, C11.2, C12.2, C13.2, C14.2, C15.2, C16.2, C17.2, C18.2, C2.2, C3.2, C4.2, C5.2, C6.2, C7.2, C8.2, C9.2, DRV_1.1 (Pin_1), DRV_1.16 (Pin_16), DRV_1.4 (Pin_4), DRV_2.1 (Pin_1), DRV_2.16 (Pin_16), DRV_2.4 (Pin_4), DRV_3.1 (Pin_1), DRV_3.16 (Pin_16), DRV_3.4 (Pin_4), DRV_4.1 (Pin_1), DRV_4.16 (Pin_16), DRV_4.4 (Pin_4), DRV_5.1 (Pin_1), DRV_5.16 (Pin_16), DRV_5.4 (Pin_4), DRV_6.1 (Pin_1), DRV_6.16 (Pin_16), DRV_6.4 (Pin_4)
- no-connect marks 0 -> 6

Commit message: Started PCB layout for test board
Parts:
- DRV_1, DRV_2, DRV_3, DRV_4, DRV_5, DRV_6: footprint PinSocket_2x08_P2.54mm -> Robot:TMC5160T_Pro_V1.0_Breakout
- J1: footprint (none) -> Robot:TMC5160T_Pro_V1.0_Breakout
Changed lines of the file:
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@@
 			)
 		)
-		(property "Footprint" ""
+		(property "Footprint" "Robot:TMC5160T_Pro_V1.0_Breakout"
 			(at 35.56 76.2 0)
 			(effects
@@
 			)
 		)
-		(property "Footprint" "PinSocket_2x08_P2.54mm"
+		(property "Footprint" "Robot:TMC5160T_Pro_V1.0_Breakout"
 			(at 63.754 59.944 0)
 			(effects
@@
 			)
 		)
-		(property "Footprint" "PinSocket_2x08_P2.54mm"
+		(property "Footprint" "Robot:TMC5160T_Pro_V1.0_Breakout"
 			(at 139.954 110.744 0)
 			(effects
@@
 			)
 		)
-		(property "Footprint" "PinSocket_2x08_P2.54mm"
+		(property "Footprint" "Robot:TMC5160T_Pro_V1.0_Breakout"
 			(at 216.154 59.944 0)
 			(effects
@@
 			)
 		)
-		(property "Footprint" "PinSocket_2x08_P2.54mm"
+		(property "Footprint" "Robot:TMC5160T_Pro_V1.0_Breakout"
 			(at 63.754 110.744 0)
 			(effects
@@
 			)
 		)
-		(property "Footprint" "PinSocket_2x08_P2.54mm"
+		(property "Footprint" "Robot:TMC5160T_Pro_V1.0_Breakout"
 			(at 216.154 110.744 0)
 			(effects
@@
 			)
 		)
-		(property "Footprint" "PinSocket_2x08_P2.54mm"
+		(property "Footprint" "Robot:TMC5160T_Pro_V1.0_Breakout"
 			(at 139.954 59.944 0)
 			(effects

Commit message: Updated test board
Parts:
- removed C16, C17, C18, C7, C8, C9: 100nF, Capacitor_THT:CP_Radial_D8.0mm_P2.50mm, symbol Device:C
- added J13: Screw_Terminal_01x04, TerminalBlock_Phoenix:TerminalBlock_Phoenix_MKDS-1,5-4-5.08_1x04_P5.08mm_Horizontal, symbol Connector:Screw_Terminal_01x04
- J1: footprint Robot:TMC5160T_Pro_V1.0_Breakout -> Connector_PinHeader_2.54mm:PinHeader_1x06_P2.54mm_Vertical
Connections:
- net +24V: now also J13.2 (Pin_2)
- net +3.3V: now also J13.1 (Pin_1)
- net GND: now also J13.3 (Pin_3), J13.4 (Pin_4)

Commit message: Cleaned up test board
Parts:
- renumbered C13 to C10, C14 to C11, C15 to C12, C10 to C7, C11 to C8, C12 to C9, J13 to J1, J9 to J10, J10 to J11, J11 to J12, J12 to J13, J1 to J2, J2 to J3, J3 to J4, J4 to J5, J5 to J6, J6 to J7, J7 to J8, J8 to J9
Connections:
- net +24V: now also J1.1 (Pin_1); no longer J1.2 (Pin_2)
- net +3.3V: now also J1.3 (Pin_3); no longer J1.1 (Pin_1)
- net GND: now also J1.2 (Pin_2); no longer J1.3 (Pin_3)
Other:
- note added: "Drivers / Connectors"
- note added: "Supply"
- company: (none) -> github.com/EmanuelKaefer/Open-robot-arm
- title: (none) -> Test board

Commit message: Fixed the whole test thing
Parts:
- removed J10, J12, J2, J4, J6, J8: Conn_01x06_Pin, Connector_PinHeader_2.54mm:PinHeader_1x06_P2.54mm_Vertical, symbol Connector:Conn_01x06_Pin
- added D1: D_TVS, Diode_THT:D_DO-201AD_P15.24mm_Horizontal, symbol Device:D_TVS
- added J1, J12, J13, J14, J6, J7, J8: Conn_01x03_Pin, Connector_PinHeader_2.54mm:PinHeader_1x03_P2.54mm_Vertical, symbol Connector:Conn_01x03_Pin
- added R1, R10, R11, R12, R2, R3, R4, R5, R6, R7, R8, R9: 0Ohm, Resistor_THT:R_Axial_DIN0207_L6.3mm_D2.5mm_P10.16mm_Horizontal, symbol Device:R
- renumbered J11 to J10, J13 to J11, J1 to J2, J5 to J4, J7 to J5
Connections:
- net +24V: now also D1.1 (A1)
- net GND: now also D1.2 (A2)
- net at DRV_2.3 (Pin_3): now also R2.2
- net SCK: now reaches DRV_2.5 (Pin_5)
- net SCK: now also DRV_1.5 (Pin_5), DRV_3.5 (Pin_5), DRV_4.5 (Pin_5), DRV_5.5 (Pin_5), DRV_6.5 (Pin_5), J1.2 (Pin_2)
- net at DRV_2.7 (Pin_7): now also J7.1 (Pin_1)
- net at DRV_2.9 (Pin_9): now also R5.2
- net at DRV_2.13 (Pin_13): now also J7.2 (Pin_2)
- net at DRV_2.15 (Pin_15): now also J7.3 (Pin_3)
- net at DRV_4.3 (Pin_3): now also R7.2
- net at DRV_4.7 (Pin_7): now also J12.1 (Pin_1)
- net at DRV_4.9 (Pin_9): now also R10.2
- net at DRV_4.13 (Pin_13): now also J12.2 (Pin_2)
- net at DRV_4.15 (Pin_15): now also J12.3 (Pin_3)
- net at DRV_3.3 (Pin_3): now also R3.2
- net at DRV_3.7 (Pin_7): now also J8.1 (Pin_1)
- net at DRV_3.9 (Pin_9): now also R6.2
- net at DRV_3.13 (Pin_13): now also J8.2 (Pin_2)
- net at DRV_3.15 (Pin_15): now also J8.3 (Pin_3)
- net at DRV_1.3 (Pin_3): now also R1.2
- net at DRV_1.7 (Pin_7): now also J6.1 (Pin_1)
- net at DRV_1.9 (Pin_9): now also R4.2
- net at DRV_1.13 (Pin_13): now also J6.2 (Pin_2)
- net at DRV_1.15 (Pin_15): now also J6.3 (Pin_3)
- net at DRV_6.3 (Pin_3): now also R9.2
- net at DRV_6.7 (Pin_7): now also J14.1 (Pin_1)
- net at DRV_6.9 (Pin_9): now also R12.2
- net at DRV_6.13 (Pin_13): now also J14.2 (Pin_2)
- net at DRV_6.15 (Pin_15): now also J14.3 (Pin_3)
- net at DRV_5.3 (Pin_3): now also R8.2
- net at DRV_5.7 (Pin_7): now also J13.1 (Pin_1)
- net at DRV_5.9 (Pin_9): now also R11.2
- net at DRV_5.13 (Pin_13): now also J13.2 (Pin_2)
- net at DRV_5.15 (Pin_15): now also J13.3 (Pin_3)
- new net MISO: J1.3 (Pin_3), R10.1, R11.1, R12.1, R4.1, R5.1, R6.1
- new net MOSI: J1.1 (Pin_1), R1.1, R2.1, R3.1, R7.1, R8.1, R9.1
Other:
- note added: "SPI"
- moved on the sheet: C11, C12, C2, C3, C5, C6, C8, C9, DRV_2, DRV_3, DRV_5, DRV_6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

Commit message: Final adjustments to test board (hopefully)
Connections:
- net MISO: now also DRV_1.9 (Pin_9), DRV_2.9 (Pin_9), DRV_3.9 (Pin_9), DRV_4.9 (Pin_9), DRV_5.9 (Pin_9), DRV_6.9 (Pin_9); no longer R10.1, R11.1, R12.1, R4.1, R5.1, R6.1
- net SCK: now also R10.1, R11.1, R12.1, R4.1, R5.1, R6.1; no longer DRV_1.5 (Pin_5), DRV_2.5 (Pin_5), DRV_3.5 (Pin_5), DRV_4.5 (Pin_5), DRV_5.5 (Pin_5), DRV_6.5 (Pin_5)
- net at R4.2: now also DRV_1.5 (Pin_5); no longer DRV_1.9 (Pin_9)
- net at R5.2: now also DRV_2.5 (Pin_5); no longer DRV_2.9 (Pin_9)
- net at R10.2: now also DRV_4.5 (Pin_5); no longer DRV_4.9 (Pin_9)
- net at R11.2: now also DRV_5.5 (Pin_5); no longer DRV_5.9 (Pin_9)
- net at R6.2: now also DRV_3.5 (Pin_5); no longer DRV_3.9 (Pin_9)
- net at R12.2: now also DRV_6.5 (Pin_5); no longer DRV_6.9 (Pin_9)
