Commit message: add MOVEIT2 and Rviz configuration

File: Software/ros2_ws/src/robot_description/urdf/robot_armV2SLDASM.urdf (robot description, URDF)
Before this commit: robot robot_armV2.SLDASM, 7 links, 6 joints
Joints:
- joint elbow_joint: limit lower=-1.5708 upper=1.5708 effort=1 velocity=1 -> lower=-1.5708 upper=1.5708 effort=1.0 velocity=1.0
- joint shoulder_joint2: limit lower=-1.5708 upper=1.5708 effort=1 velocity=1 -> lower=-1.5708 upper=1.5708 effort=1.0 velocity=1.0
- joint wrist_tilt_joint: limit lower=-2.0944 upper=1.5708 effort=1 velocity=1 -> lower=-2.0944 upper=1.5708 effort=1.0 velocity=1.0

Commit message: everythong works now wow
fixing a bug in the urdf which caused the ros_controller_node to crash right after startup, caused by the continous joints in the urdf

File: Software/ros2_ws/src/robot_description/urdf/robot_armV2SLDASM.urdf (robot description, URDF)
Before this commit: robot robot_armV2SLDASM, 7 links, 6 joints
Joints:
- joint gripper_turn_joint: limit (none) -> lower=-6.28 upper=6.28 effort=50 velocity=3.14; type continuous -> revolute
- joint shoulder_joint1: limit (none) -> lower=-6.28 upper=6.28 effort=50 velocity=3.14; type continuous -> revolute
- joint wrist_turn_joint: limit (none) -> lower=-6.28 upper=6.28 effort=50 velocity=3.14; type continuous -> revolute
